File: phased_array.kicad_sch (KiCad schematic)
At the start: 37 parts, among them U1 CUSA-T80-18-2400-TH, U10 CUSA-T80-18-2400-TH, U11 CUSA-T80-18-2400-TH, U12 CUSA-T80-18-2400-TH, U13 CUSA-T80-18-2400-TH, U14 CUSA-T80-18-2400-TH, U15 CUSA-T80-18-2400-TH, U16 CUSA-T80-18-2400-TH, U17 Tang_Nano_9k, U18 CUSA-T80-18-2400-TH, U19 CUSA-T80-18-2400-TH, U2 CUSA-T80-18-2400-TH, U20 CUSA-T80-18-2400-TH, U21 CUSA-T80-18-2400-TH, U22 CUSA-T80-18-2400-TH, U23 CUSA-T80-18-2400-TH, U24 CUSA-T80-18-2400-TH, U25 CUSA-T80-18-2400-TH, U26 CUSA-T80-18-2400-TH, U27 CUSA-T80-18-2400-TH, U28 CUSA-T80-18-2400-TH, U29 CUSA-T80-18-2400-TH, U3 CUSA-T80-18-2400-TH, U30 CUSA-T80-18-2400-TH, U31 CUSA-T80-18-2400-TH, U32 CUSA-T80-18-2400-TH, U33 CUSA-T80-18-2400-TH, U34 ULN2803A, U35 ULN2803A, U36 ULN2803A, U37 ULN2803A, U4 CUSA-T80-18-2400-TH, U5 CUSA-T80-18-2400-TH, U6 CUSA-T80-18-2400-TH, U7 CUSA-T80-18-2400-TH, U8 CUSA-T80-18-2400-TH, U9 CUSA-T80-18-2400-TH

Commit message: 1014
Parts:
- added J1: Barrel_Jack_Switch, Connector_BarrelJack:BarrelJack_Horizontal, symbol Connector:Barrel_Jack_Switch
- added J2: Conn_01x03, Connector_PinHeader_2.54mm:PinHeader_1x03_P2.54mm_Vertical, symbol Connector_Generic:Conn_01x03
- U34, U35, U36, U37: footprint (none) -> MyLibrary:DIP762W55P254L2286H480Q18N_with_solderjumper
Connections:
- net GND: now also U17. (GND), J1.1, J1.2
- net at U34.1 (I1): now also U17.69 (IOT42A/RGB_G3/HDMI_CKP)
- net at U34.2 (I2): now also U17.68 (IOT42B/RGB_G4/HDMI_CKN)
- net at U34.3 (I3): now also U17.57 (IOR13A/RGB_G5)
- net at U34.4 (I4): now also U17.56 (IOR14A/RGB_G6)
- net at U34.5 (I5): now also U17.55 (IOR14B/RGB_G7)
- net at U34.6 (I6): now also U17.54 (IOR15A/RGB_B3)
- net at U34.7 (I7): now also U17.53 (IOR15B/RGB_B4)
- net at U34.8 (I8): now also U17.51 (IOR17B/RGB_B5)
- net at U17.25 (IOB8A): now also U37.4 (I4)
- net at U17.26 (IOB8B): now also U37.3 (I3)
- net at U17.27 (IOB11A): now also U37.2 (I2)
- net at U17.28 (IOB11B): now also U37.1 (I1)
- net at U17.29 (IOB13A): now also U35.8 (I8)
- net at U17.30 (IOB13B): now also U35.7 (I7)
- net at U17.33 (IOB23A/RGB_DE): now also U35.6 (I6)
- net at U17.34 (IOB23B/RGB_VS): now also U35.5 (I5)
- net at U17.35 (IOB29A/RGB_CK): now also U35.3 (I3)
- net at U17.36 (IOB29B/TF_SCK): now also U37.5 (I5)
- net at U17.37 (IO31A/TF_MOSI): now also U37.7 (I7)
- net at U17.38 (IOB31B/TF_CS): now also U37.8 (I8)
- net at U17.39 (IOB33A/TF_MISO): now also U37.6 (I6)
- net at U17.40 (IOB33B/RGB_HS): now also U35.4 (I4)
- net at U17.41 (IOB41A/RGB_B7): now also U35.2 (I2)
- net at U17.42 (IOB41B/RGB_B6): now also U35.1 (I1)
- net at U17.70 (IOT41B/RGB_G2/HDMI_C0N): now also U36.8 (I8)
- net at U17.71 (IOT41A/RGB_R7/HDMI_D0P): now also U36.7 (I7)
- net at U17.72 (IOT39B/RGB_R6/HDMI_D1N): now also U36.6 (I6)
- net at U17.73 (IOT39A/RGB_R5/HDMI_D1P): now also U36.5 (I5)
- net at U17.74 (IOT38B/RGB_R4/HDMI_D2N): now also U36.4 (I4)
- net at U17.75 (IOT38A/RGB_R3/HDMI_D2P): now also U36.3 (I3)
- net at U17.76 (IOT37B/SPILCD_CK): now also U36.2 (I2)
- net at U17.77 (IOT37A/SPILCD_MO): now also U36.1 (I1)
- net at U1.2, U10.2, U11.2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: now also U18.2, U19.2, U20.2, U21.2, U22.2, U23.2, U24.2, U25.2, U26.2, U27.2, U28.2, U29.2, U30.2, U31.2, U32.2, U33.2, J2.2 (Pin_2)
- removed net VCC: U16.1, U18.2, U19.2, U20.2, U21.2, U22.2, U23.2, U24.2, U25.2, U26.2, U27.2, U28.2, U29.2, U30.2, U31.2, U32.2, U33.2, U37.18 (O1)
- new net: U16.1, U37.18 (O1)
- new net: J1.3, J2.1 (Pin_1)
- new net +3.3V: J2.3 (Pin_3), U17. (GND)
- new net +5V: U17. (GND)
Other:
- moved on the sheet: U17

Commit message: 1015
Parts:
- U1, U10, U11, U12, U13, U14, U15, U16, U18, U19, U2, U20, U21, U22, U23, U24, U25, U26, U27, U28, U29, U3, U30, U31, U32, U33, U4, U5, U6, U7, U8, U9: footprint CUSAT80182400TH -> SamacSys_Parts:CUSAT80182400TH
- U17: footprint Custom Library:Tang Nano 9K -> MyLibrary:Tang Nano 9K
Connections:
- net +3.3V: now also U17.25 (3V3); no longer J2.3 (Pin_3), U17. (GND)
- net +5V: now also J2.3 (Pin_3), U17.31 (5V); no longer U17. (GND)
- net GND: now also U17.26 (GND); no longer U17. (GND)
- net at U34.1 (I1): now also U17.24 (IOT42A/RGB_G3/HDMI_CKP/69); no longer U17.69 (IOT42A/RGB_G3/HDMI_CKP)
- net at U34.2 (I2): now also U17.23 (IOT42B/RGB_G4/HDMI_CKN/68); no longer U17.68 (IOT42B/RGB_G4/HDMI_CKN)
- net at U34.3 (I3): now also U17.22 (IOR13A/RGB_G5/57); no longer U17.57 (IOR13A/RGB_G5)
- net at U34.4 (I4): now also U17.21 (IOR14A/RGB_G6/56); no longer U17.56 (IOR14A/RGB_G6)
- net at U34.5 (I5): now also U17.20 (IOR14B/RGB_G7/55); no longer U17.55 (IOR14B/RGB_G7)
- net at U34.6 (I6): now also U17.19 (IOR15A/RGB_B3/54); no longer U17.54 (IOR15A/RGB_B3)
- net at U34.7 (I7): now also U17.18 (IOR15B/RGB_B4/53); no longer U17.53 (IOR15B/RGB_B4)
- net at U34.8 (I8): now also U17.17 (IOR17B/RGB_B5/51); no longer U17.51 (IOR17B/RGB_B5)
- net at U37.4 (I4): now also U17.5 (IOB8A/25); no longer U17.25 (IOB8A)
- net at U37.3 (I3): now also U17.6 (IOB8B/26); no longer U17.26 (IOB8B)
- net at U17.27 (IOB15B/RGB_TOUCH_XR/32): no longer U37.2 (I2)
- net at U17.28 (IOB15A/RGB_TOUCH_YD/31): no longer U37.1 (I1)
- net at U17.29 (IOR24A/SPILCD_RS/49): no longer U35.8 (I8)
- net at U35.7 (I7): now also U17.10 (IOB13B/30); no longer U17.30 (IOB13B)
- net at U17.32 (IOT41B/RGB_G2/HDMI_C0N/70): now also U36.8 (I8)
- net at U35.6 (I6): now also U17.11 (IOB23A/RGB_DE/33); no longer U17.33 (IOB23A/RGB_DE)
- net at U35.5 (I5): now also U17.12 (IOB23B/RGB_VS/34); no longer U17.34 (IOB23B/RGB_VS)
- net at U35.3 (I3): now also U17.14 (IOB29A/RGB_CK/35); no longer U17.35 (IOB29A/RGB_CK)
- net at U17.36 (IOT38B/RGB_R4/HDMI_D2N/74): now also U36.4 (I4); no longer U37.5 (I5)
- net at U37.7 (I7): now also U17.2 (IO31A/TF_MOSI/37); no longer U17.37 (IO31A/TF_MOSI)
- net at U37.8 (I8): now also U17.1 (IOB31B/TF_CS/38); no longer U17.38 (IOB31B/TF_CS)
- net at U37.6 (I6): now also U17.3 (IOB33A/TF_MISO/39); no longer U17.39 (IOB33A/TF_MISO)
- net at U35.4 (I4): now also U17.13 (IOB33B/RGB_HS/40); no longer U17.40 (IOB33B/RGB_HS)
- net at U35.2 (I2): now also U17.15 (IOB41A/RGB_B7/41); no longer U17.41 (IOB41A/RGB_B7)
- net at U35.1 (I1): now also U17.16 (IOB41B/RGB_B6/42); no longer U17.42 (IOB41B/RGB_B6)
- net at U36.7 (I7): now also U17.33 (IOT41A/RGB_R7/HDMI_D0P/71); no longer U17.71 (IOT41A/RGB_R7/HDMI_D0P)
- net at U36.6 (I6): now also U17.34 (IOT39B/RGB_R6/HDMI_D1N/72); no longer U17.72 (IOT39B/RGB_R6/HDMI_D1N)
- net at U36.5 (I5): now also U17.35 (IOT39A/RGB_R5/HDMI_D1P/73); no longer U17.73 (IOT39A/RGB_R5/HDMI_D1P)
- net at U36.3 (I3): now also U17.37 (IOT38A/RGB_R3/HDMI_D2P/75); no longer U17.75 (IOT38A/RGB_R3/HDMI_D2P)
- net at U36.2 (I2): now also U17.38 (IOT37B/SPILCD_CK/76); no longer U17.76 (IOT37B/SPILCD_CK)
- net at U36.1 (I1): now also U17.39 (IOT37A/SPILCD_MO/77); no longer U17.77 (IOT37A/SPILCD_MO)
- new net: U17.4 (IOB29B/TF_SCK/36), U37.5 (I5)
- new net: U17.7 (IOB11A/27), U37.2 (I2)
- new net: U17.8 (IOB11B/28), U37.1 (I1)
- new net: U17.9 (IOB13A/29), U35.8 (I8)
