File: phased_array.kicad_pcb (KiCad board)
At the start: 2 copper layers, 99.6 x 99.6 mm, 39 parts, among them J1 Barrel_Jack_Switch, J2 Conn_01x03, U1 CUSA-T80-18-2400-TH, U10 CUSA-T80-18-2400-TH, U11 CUSA-T80-18-2400-TH, U12 CUSA-T80-18-2400-TH, U13 CUSA-T80-18-2400-TH, U14 CUSA-T80-18-2400-TH, U15 CUSA-T80-18-2400-TH, U16 CUSA-T80-18-2400-TH, U17 Tang_Nano_9k, U18 CUSA-T80-18-2400-TH, U19 CUSA-T80-18-2400-TH, U2 CUSA-T80-18-2400-TH, U20 CUSA-T80-18-2400-TH, U21 CUSA-T80-18-2400-TH, U22 CUSA-T80-18-2400-TH, U23 CUSA-T80-18-2400-TH, U24 CUSA-T80-18-2400-TH, U25 CUSA-T80-18-2400-TH, U26 CUSA-T80-18-2400-TH, U27 CUSA-T80-18-2400-TH, U28 CUSA-T80-18-2400-TH, U29 CUSA-T80-18-2400-TH, U3 CUSA-T80-18-2400-TH, U30 CUSA-T80-18-2400-TH, U31 CUSA-T80-18-2400-TH, U32 CUSA-T80-18-2400-TH, U33 CUSA-T80-18-2400-TH, U34 ULN2803A, U35 ULN2803A, U36 ULN2803A, U37 ULN2803A, U4 CUSA-T80-18-2400-TH, U5 CUSA-T80-18-2400-TH, U6 CUSA-T80-18-2400-TH, U7 CUSA-T80-18-2400-TH, U8 CUSA-T80-18-2400-TH, U9 CUSA-T80-18-2400-TH

Commit message: 1015
Parts:
- U11, U12, U13, U14, U15, U16: moved to B.Cu
- moved U25 360.8 mm to (468.4, 27.1)
- moved U24 345.0 mm to (454.2, 25.6)
- moved U32 333.6 mm to (462.8, 66.2)
- moved U33 310.9 mm to (439.4, 68.2)
- moved U9 307.6 mm to (372.4, 117.0)
- moved U20 305.4 mm to (385.6, 27.6)
- moved U27 303.4 mm to (411.0, 69.2)
- moved U21 289.9 mm to (363.2, 27.6)
- moved U28 283.7 mm to (387.6, 68.2)
- moved U10 283.0 mm to (351.0, 117.1)
- moved U22 281.0 mm to (345.4, 27.1)
- moved U19 274.0 mm to (356.1, 19.9)
- moved U29 260.6 mm to (359.2, 69.6)
- moved U18 238.6 mm to (324.1, 18.9)
- moved U26 226.7 mm to (335.8, 67.7)
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